File: uSomIQ-daughterboards/serial/serial.sch (EAGLE design)
At the start: 0 parts

Commit message: Add uSomIQ-AM334x to library
Parts:
- added U$3: USOMIQ-AM335X, connectors:USOMIQ-AM335X
Changed lines of the file:
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@@
 <part name="U$1" library="titleblock" deviceset="REDLINE-TITLEBLOCK" device=""/>
 <part name="U$2" library="titleblock" deviceset="REDLINE-TITLEBLOCK" device=""/>
+<part name="U$3" library="connectors" deviceset="USOMIQ-AM335X" device=""/>
 </parts>
 <sheets>
@@
 <instances>
 <instance part="U$2" gate="G$1" x="0" y="0"/>
+<instance part="U$3" gate="G$1" x="55.88" y="91.44"/>
 </instances>
 <busses>

Commit message: Add power supply and RTC
Parts:
- added C1, C2: 4.7uF, 50V, rcl:C-USC1210
- added C3: 0.01uF, 50V, rcl:C-USC0603
- added C4: 0.1uF, 50V, rcl:C-USC0603
- added C5: 5600pF, 25V, rcl:C-USC0603
- added C6: 330pF, 50V, rcl:C-USC0603
- added C7, C8: 47uF, 16V, rcl:C-USC2220K
- added C9: 1uF, 16V, rcl:C-USC0603
- added D1, D2, D5: B360B, diode:SCHOTTKY-DIODESMD
- added D3, D4: 47V, diode:ZENER-DIODESMB
- added IC1: DS3231/SO, adafruit:DS3231/SO
- added L1: 27uH, 4.3A, power-supplies:L-US
- added LED1: (no value), led:LEDSML0603
- added R1: 384K, rcl:R-US_R0603
- added R2: 69.8K, rcl:R-US_R0603
- added R3: 412K, rcl:R-US_R0603
- added R4: 53.6K, rcl:R-US_R0603
- added R5, R7: 10K, rcl:R-US_R0603
- added R6: 11K, rcl:R-US_R0603
- added R8, R9: 100, rcl:R-US_R0603
- added U$4: TPS54260, power-supplies:TPS54260
- added U$7: (no value), adafruit:CR1220THM
Connections:
- new net GND: C1.2, C2.2, C3.2, C5.2, C6.2, C7.2, C8.2, C9.2, D3.A, D4.A, D5.A, IC1.GND, LED1.C, R2.1, R3.1, R5.1, U$3.GND@0, U$3.GND@1, U$3.GND@2, U$3.GND@3, U$4.GND, U$4.PAD, U$7.-
- new net I2C0_SCL: IC1.SCL
- new net I2C0_SDA: IC1.SDA
- new net N$1: C1.1, C2.1, D1.C, D3.C, U$4.VIN
- new net N$10: C6.1, R6.2, U$4.COMP
- new net N$11: C5.1, R6.1
- new net N$12: IC1.VBAT, U$7.+
- new net N$2: C3.1, U$4.SS/TR
- new net N$3: D2.C, D4.C, R1.1
- new net N$4: R1.2, R2.2, U$4.EN
- new net N$5: R3.2, U$4.RT/CLK
- new net N$6: C4.1, U$4.BOOT
- new net N$7: C4.2, D5.C, L1.1, U$4.PH
- new net N$8: IC1.32KHZ, R9.2
- new net N$9: R4.1, R5.2, U$4.VSNS
- new net RESET: R8.1
- new net RTC_32KHZ: R9.1
- new net VBATT: D1.A
- new net VDD: C7.1, C8.1, C9.1, IC1.VCC, L1.2, R4.2, R7.2
- new net VDD_PGOOD: LED1.A, R7.1, R8.2, U$4.PWRGD
- new net VIGN: D2.A
Other:
- note added: "2. SOM Header"
- note added: "3. RTC and EEPROM"
- note added: "Based on TI application design, TIDA-00322"
- note added: "RTC"
- note added: "TODO: Need to revisit this! Backfeed"
- note added: "VDD_PGOOD is an open-drain output that asserts when power supply is out of spec"

Commit message: Add serial port connectors
Parts:
- added U$6: 83611-9006, connectors:83611-9006
- added U$8, U$9: 189-009-613R571, connectors:189-009-613R571
Connections:
- new net CAN_H: U$6.5
- new net CAN_L: U$6.6
- new net ETH_RX+: U$6.3
- new net ETH_RX-: U$6.4
- new net ETH_TX+: U$6.1
- new net ETH_TX-: U$6.2
- new net SP0-1PPS: U$8G$1.1
- new net SP0-RX: U$8G$1.2
- new net SP0-TX: U$8G$1.3
- new net SP1-1PPS: U$8G$2.1
- new net SP1-RX: U$8G$2.2
- new net SP1-TX: U$8G$2.3
- new net SP2-1PPS: U$9G$1.1
- new net SP2-RX: U$9G$1.2
- new net SP2-TX: U$9G$1.3
- new net SP3-1PPS: U$9G$2.1
- new net SP3-RX: U$9G$2.2
- new net SP3-TX: U$9G$2.3
- net GND: now also U$6.9, U$6.MOUNT@1, U$6.MOUNT@2, U$8G$1.5, U$8G$1.MOUNT@0, U$8G$1.MOUNT@1, U$8G$2.5, U$8G$2.MOUNT@0, U$8G$2.MOUNT@1, U$9G$1.5, U$9G$1.MOUNT@0, U$9G$1.MOUNT@1, U$9G$2.5, U$9G$2.MOUNT@0, U$9G$2.MOUNT@1
- net VBATT: now also U$6.7
- net VIGN: now also U$6.8
Other:
- note added: "Connectors"
- note added: "Daughterboard Specific Connectors"
- note added: "Most nodes should implement 100Mb ethernet CAN is also available for very basic, low cost nodes"
- note added: "Primary connector"

Commit message: Add RS232 transcievers
Parts:
- added C10, C11, C12, C13, C14, C17, C18, C19, C20, C21: 0.1uF, resistor:C-USC0603
- added C15, C16, C22, C23: 10uF, resistor:C-USC0603
- added R10, R11, R12, R13, R14, R15, R16, R17: 1k, resistor:R-US_R0603
- added TP1, TP2, TP3, TP4: TPB1,27, testpad:TPB1,27
- added U$10, U$11: ADM3311E, misc-ics:ADM3311E
Connections:
- new net +3V3: C10.2, C15.1, C16.1, C17.2, C22.1, C23.1, R16.2, R17.2, U$10.VCC, U$11.VCC, U$3.P2-6, U$3.P2-8
- new net +5V: C7.1, C8.1, L1.2, R4.2, U$3.P2-2, U$3.P2-4
- new net N$13: C10.1, U$10.V+
- new net N$14: C17.1, U$11.V+
- new net N$15: C11.1, U$10.C2+
- new net N$16: C11.2, U$10.C2-
- new net N$17: R10.2, U$10.T3IN
- new net N$18: TP1.TP, U$10.R5OUT
- new net N$19: TP2.TP, U$10.T3OUT
- new net N$20: R11.2, U$10.R5IN
- new net N$21: R12.2, U$10.SD
- new net N$22: C12.1, U$10.C1+
- new net N$23: C12.2, U$10.C1-
- new net N$24: C13.2, U$10.V-
- new net N$25: C18.1, U$11.C2+
- new net N$26: C14.2, U$10.C3-
- new net N$27: C14.1, U$10.C3+
- new net N$28: C18.2, U$11.C2-
- new net N$29: R13.2, U$11.T3IN
- new net N$30: TP3.TP, U$11.R5OUT
- new net N$31: TP4.TP, U$11.T3OUT
- new net N$32: R14.2, U$11.R5IN
- new net N$33: R15.2, U$11.SD
- new net N$34: C19.1, U$11.C1+
- new net N$35: C19.2, U$11.C1-
- new net N$36: C20.2, U$11.V-
- new net N$37: C21.2, U$11.C3-
- new net N$38: C21.1, U$11.C3+
- new net N$40: R7.2
- new net SP0_1PPS: U$10.R2IN, U$11.R2IN
- new net SP0_RX: U$10.R1IN, U$11.R1IN
- new net SP0_TX: U$10.T1OUT, U$11.T1OUT
- new net SP1_1PPS: U$10.R4IN, U$11.R4IN
- new net SP1_RX: U$10.R3IN, U$11.R3IN
- new net SP1_TX: U$10.T2OUT, U$11.T2OUT
- new net UART0_1PPS: U$10.R2OUT, U$11.R2OUT, U$3.P2-33
- new net UART0_RX: U$10.R1OUT, U$11.R1OUT, U$3.P2-29
- new net UART0_TX: U$10.T1IN, U$11.T1IN, U$3.P2-31
- new net UART1_1PPS: U$10.R4OUT, U$11.R4OUT, U$3.P2-40
- new net UART1_RX: U$10.R3OUT, U$11.R3OUT, U$3.P2-37
- new net UART1_TX: U$10.T2IN, U$11.T2IN, U$3.P2-39
- new net UART2_1PPS: U$3.P2-50
- new net UART2_RX: U$3.P2-49
- new net UART2_TX: U$3.P2-47
- new net UART3_1PPS: U$3.P2-46
- new net UART3_RX: U$3.P2-41
- new net UART3_TX: U$3.P2-43
- new net XCVR_EN: R16.1, R17.1, U$10.EN, U$11.EN
- net GND: now also C13.1, C15.2, C16.2, C20.1, C22.2, C23.2, R10.1, R11.1, R12.1, R13.1, R14.1, R15.1, U$10.GND, U$11.GND, U$3.P2-1, U$3.P2-3
- net I2C0_SCL: now also U$3.P2-12
- net I2C0_SDA: now also U$3.P2-10
- net VDD: no longer C7.1, C8.1, L1.2, R4.2, R7.2
Other:
- note added: "1.5/cm"
- note added: "1.75/cm"
- note added: "2.0/cm"
- note added: "24AWG"
- note added: "BK"
- note added: "CAN_H"
- note added: "CAN_L"
- note added: "Cable Construction"
- note added: "Color"
- note added: "Conductor"
- note added: "ETH_RX+"
- note added: "ETH_RX-"
- note added: "ETH_TX+"
- note added: "ETH_TX-"
- note added: "GN"
- note added: "GN/YL"
- note added: "GND"
- note added: "Gauge"
- note added: "OR"
- note added: "PK"
- note added: "RD"
- note added: "Shield TBD"
- note added: "Twists"
- note added: "VBATT"
- note added: "VIGN"
- note added: "WT/GN"
- note added: "WT/OR"
- note added: "YL/VT"

Commit message: Update libraries, add power supply monitoring
Parts:
- removed C1: 4.7uF, 50V, rcl:C-USC1210
- removed D2: B360B, diode:SCHOTTKY-DIODESMD
- removed LED1: (no value), led:LEDSML0603
- removed R1: 384K, rcl:R-US_R0603
- removed R2: 69.8K, rcl:R-US_R0603
- removed R7: 10K, rcl:R-US_R0603
- removed R8: 100, rcl:R-US_R0603
- added C201: 0.1uF, rcl:C-USC1210
- added C202: 4.7uF, 50V, rcl:C-USC1210
- added C210, C211: 0.1uF, rcl:C-USC0603
- added D202, D207: BAS40, diode:BAS40
- added D203: B360B, diode:SCHOTTKY-DIODESMD
- added D208, D209: 1.8V, diode:ZENER-DIODESMB
- added LED201, LED301, LED302: (no value), led:LEDSML0603
- added R201: NL, rcl:R-US_R0603
- added R202, R301, R302: 10K, rcl:R-US_R0603
- added R203: 384K, rcl:R-US_R0603
- added R204: 69.8K, rcl:R-US_R0603
- added R209, R210: 20K, rcl:R-US_R0603
- added R211, R212: 1K, rcl:R-US_R0603
- added R405: 100, rcl:R-US_R0603
- added X301: MINI-USB-UX60-MB-5ST, con-hirose:MINI-USB-UX60-MB-5ST
- renumbered C10 to C403, C11 to C402, C12 to C405, C13 to C407, C14 to C408, C15 to C401, C16 to C404, C17 to C411, C18 to C410, C19 to C413, C2 to C203, C20 to C414, C21 to C415, C22 to C409, C23 to C412, C3 to C204, C4 to C205, C5 to C206, C6 to C207, C7 to C208, C8 to C209, C9 to C406, D1 to D201, D3 to D204, D4 to D205, D5 to D206, IC1 to IC401, L1 to L201, R10 to R402, R11 to R403, R12 to R406, R13 to R408, R14 to R409, R15 to R410, R16 to R401, R17 to R407, R3 to R205, R4 to R207, R5 to R208, R6 to R206, R9 to R404, U$10 to U401, U$11 to U402, U$3 to P301, U$4 to U201, U$6 to P102, U$7 to B401, U$8 to P101, U$9 to P103
Connections:
- removed net N$1: C1.1, C203.1, D201.C, D204.C, U201.VIN
- removed net SP0-1PPS: P101G$1.1
- removed net SP0-RX: P101G$1.2
- removed net SP0-TX: P101G$1.3
- removed net SP1-1PPS: P101G$2.1
- removed net SP1-RX: P101G$2.2
- removed net SP1-TX: P101G$2.3
- removed net SP2-1PPS: P103G$1.1
- removed net SP2-RX: P103G$1.2
- removed net SP2-TX: P103G$1.3
- removed net SP3-1PPS: P103G$2.1
- removed net SP3-RX: P103G$2.2
- removed net SP3-TX: P103G$2.3
- removed net VDD: C406.1, IC401.VCC
- new net ADC_VBATT: C211.1, D209.C, P301.P2-13, R210.2, R212.2
- new net ADC_VIGN: C210.1, D208.C, P301.P2-11, R209.2, R211.2
- new net LED_ETH_100MB: P301.P2-67, R301.2
- new net LED_ETH_ACTIVE: P301.P2-69, R302.2
- new net N$39: IC401./RST, R405.2
- new net N$42: D207.C, R209.1
- new net PWR_EN: D202.A, P301.P2-38
- new net RTC_RST: R405.1
- new net SP2_1PPS: P103G$1.1, U402.R2IN
- new net SP2_RX: P103G$1.2, U402.R1IN
- new net SP2_TX: P103G$1.3, U402.T1OUT
- new net SP3_1PPS: P103G$2.1, U402.R4IN
- new net SP3_RX: P103G$2.2, U402.R3IN
- new net SP3_TX: P103G$2.3, U402.T2OUT
- new net USB_D+: P301.P2-61, X301.3
- new net USB_D-: P301.P2-63, X301.2
- new net VBATT_PROTECTED: C201.1, C202.1, C203.1, D201.C, D204.C, R210.1, U201.VIN
- new net VDD_PGOOD1: LED301.A, R301.1
- new net VDD_PGOOD2: LED302.A, R302.1
- net +3V3: now also C406.1, IC401.VCC
- net ETH_RX+: now also P301.P2-62
- net ETH_RX-: now also P301.P2-64, P301.P2-70
- net ETH_TX+: now also P301.P2-68
- net GND: now also C201.2, C202.2, C210.2, C211.2, D208.A, D209.A, LED201.C, LED301.C, LED302.C, P301.P2-27, P301.P2-59, P301.P2-60, P301.P2-65, P301.P2-66, P301.P2-9, P301.P3-21, P301.P3-22, P301.P3-59, P301.P3-65, R204.1, R211.1, R212.1, X301.5; no longer C1.2, LED1.C, R2.1
- net N$3: now also D203.C, R203.1; no longer D2.C, R1.1
- net N$4: now also R203.2, R204.2; no longer R1.2, R2.2
- net N$40: now also R202.2; no longer R7.2
- net RESET: now also R201.1; no longer R8.1
- net SP0_1PPS: now also P101G$1.1; no longer U402.R2IN
- net SP0_RX: now also P101G$1.2; no longer U402.R1IN
- net SP0_TX: now also P101G$1.3; no longer U402.T1OUT
- net SP1_1PPS: now also P101G$2.1; no longer U402.R4IN
- net SP1_RX: now also P101G$2.2; no longer U402.R3IN
- net SP1_TX: now also P101G$2.3; no longer U402.T2OUT
- net UART0_1PPS: no longer U402.R2OUT
- net UART0_RX: no longer U402.R1OUT
- net UART0_TX: no longer U402.T1IN
- net UART1_1PPS: no longer U402.R4OUT
- net UART1_RX: no longer U402.R3OUT
- net UART1_TX: no longer U402.T2IN
- net UART2_1PPS: now also U402.R2OUT
- net UART2_RX: now also U402.R1OUT
- net UART2_TX: now also U402.T1IN
- net UART3_1PPS: now also U402.R4OUT
- net UART3_RX: now also U402.R3OUT
- net UART3_TX: now also U402.T2IN
- net VDD_PGOOD: now also LED201.A, R201.2, R202.1; no longer LED1.A, R7.1, R8.2
- net VIGN: now also D203.A, D207.A; no longer D2.A
Other:
- note added: "Monitor VIGN through dedicated feed so we don't get backfeed from PWR_EN in our measurement"

Commit message: Start to place serial daughterboard power supply
Parts:
- removed C203: 4.7uF, 50V, rcl:C-USC1210
- removed C208: 47uF, 16V, rcl:C-USC2220K
- removed D203: B360B, diode:SCHOTTKY-DIODESMD
- removed R201: NL, rcl:R-US_R0603
- added D1: BAS40, diode:BAS40
- added TP5, TP6: TPB1,27, testpad:TPB1,27
- D205: device diode:ZENER-DIODESMB -> diode:ZENER-DIODESOT23
Connections:
- removed net N$40: R202.2
- removed net RESET: R201.1
- removed net RTC_32KHZ: R404.1
- removed net RTC_RST: R405.1
- new net N$1: R404.1, TP5.TP
- new net N$41: R405.1, TP6.TP
- net +5V: now also R202.2; no longer C208.1
- net ETH_RX-: no longer P301.P2-70
- net ETH_TX-: now also P301.P2-70
- net GND: no longer C203.2, C208.2
- net N$3: now also D1.C; no longer D203.C
- net N$4: now also D202.C
- net VBATT_PROTECTED: no longer C203.1
- net VDD_PGOOD: no longer R201.2
- net VIGN: now also D1.A; no longer D203.A
Other:
- note removed: "TODO: Need to revisit this! Backfeed"
